File: SI5351_broadband_comb_generatror.kicad_pcb (KiCad board)
At the start: 4 copper layers, 150 x 75 mm, 111 parts, among them J1 Conn_Coaxial_Small, J10 Conn_01x06_Socket, J11 RFShield_TwoPieces, J2 RFShield_TwoPieces, J3 Barrel_Jack_Switch, J4 Conn_Coaxial_Small, J5 Conn_01x10_Pin, J6 Conn_01x06_Socket, J7 USB_B, J8 AVR-ISP-6, J9 Conn_Coaxial_Small, SW1 SW_SP5T_NR01105, U1 ISL3280ExHZ, U10 ATmega328PB-A, U11 FT232RL, U12 WE-TVS-82400102, U13 PAT1220-C-3DB, U2 PHA-13HLN+, U4 KT2520K-T, U5 Si5351C-B-GM, U6 PHA-13HLN+, U7 PAT1220-C-3DB, U8 AMS1117-3.3, U9 L7809, Y1 ECS-2520MV-xxx-xx

Commit message: weiter layoutet
Parts:
- moved C10 99.1 mm to (151.8, 81.8), turned to 180 degrees
- moved U4 5.48 mm to (152.5, 84.8), turned to 0 degrees
- moved C1 3.69 mm to (157.0, 82.8)
- moved C2 3.20 mm to (155.0, 82.8), turned to 90 degrees
- moved R1 2.00 mm to (160.5, 82.2), turned to 180 degrees
- moved R3 1.77 mm to (149.5, 84.8), turned to -90 degrees
- moved FB1 1.25 mm to (151.8, 79.5)
- moved R2 1.00 mm to (151.0, 92.5)
Routing:
- net /Comb_Generator/3V3D: track 0.00 -> 15.9 mm
- net /Comb_Generator/INTR: track 17.9 -> 21.9 mm
- net Net-(U5-CLK0): track 0.00 -> 2.96 mm
- net /Comb_Generator/10MHz_IN: track 0.00 -> 2.67 mm
- net Net-(U5-VDDOA): track 13.8 -> 16.4 mm, vias 0 -> 2
- net Net-(U4-OUT): track 0.00 -> 2.61 mm
- net Net-(U5-CLK1): track 0.00 -> 2.21 mm
- net Net-(U1-RO): track 0.00 -> 2.16 mm

Commit message: es wird langsam...
Parts:
- added C47: 100n, Capacitor_SMD:C_0805_2012Metric_Pad1.18x1.45mm_HandSolder, F.Cu at (175.3, 115.6)
- added C48: 100n, Capacitor_SMD:C_0805_2012Metric_Pad1.18x1.45mm_HandSolder, F.Cu at (186.3, 103.1)
- added C49: 100n, Capacitor_SMD:C_0805_2012Metric_Pad1.18x1.45mm_HandSolder, F.Cu at (179.3, 61.0)
- added C50: 100n, Capacitor_SMD:C_0805_2012Metric_Pad1.18x1.45mm_HandSolder, F.Cu at (186.1, 60.0)
- added H1: MountingHole_Pad, MountingHole:MountingHole_3.2mm_M3_Pad_Via, F.Cu at (105.0, 55.0)
- added H2: MountingHole_Pad, MountingHole:MountingHole_3.2mm_M3_Pad_Via, F.Cu at (215.0, 55.0)
- added H3: MountingHole_Pad, MountingHole:MountingHole_3.2mm_M3_Pad_Via, F.Cu at (215.0, 120.0)
- added H4: MountingHole_Pad, MountingHole:MountingHole_3.2mm_M3_Pad_Via, F.Cu at (105.0, 120.0)
- J1: moved to F.Cu
- J11, J2: footprint RF_Shielding:Wuerth_36103305_30x30mm -> RF_Shielding:Wuerth_3670473_47.3x23.3
- moved C36 141.6 mm to (185.9, 115.0), turned to 90 degrees
- moved R7 138.2 mm to (187.9, 115.0), turned to -90 degrees
- moved R4 133.8 mm to (180.2, 112.0)
- moved C35 131.3 mm to (180.2, 103.1), turned to 90 degrees
- moved C42 129.9 mm to (184.2, 103.1), turned to 90 degrees
- moved C31 129.6 mm to (198.6, 69.1), turned to 180 degrees
- moved R8 129.1 mm to (177.3, 115.6), turned to -90 degrees
- moved C27 127.8 mm to (173.9, 110.0)
- moved C33 126.2 mm to (176.9, 111.0), turned to -90 degrees
- moved L5 125.9 mm to (184.2, 107.0), turned to -90 degrees
- moved C44 125.4 mm to (182.2, 103.1), turned to 90 degrees
- moved L3 124.3 mm to (192.7, 69.1)
- moved C9 123.6 mm to (189.8, 70.2), turned to 90 degrees
- moved RV2 123.5 mm to (181.6, 115.6), turned to 180 degrees
- moved C6 122.7 mm to (189.8, 58.5)
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Connections:
- C26 pad 2: GNDA -> GND
- C27 pad 1: Net-(U5-CLK1) -> /Comb_Generator/CLK0
- C32 pad 2: GNDA -> GND
- C35 pad 2: GNDA -> GND
- C36 pad 2: GNDA -> GND
- C41 pad 1: GNDA -> GND
- C42 pad 2: GNDA -> GND
- C44 pad 2: GNDA -> GND
- C5 pad 2: GNDA -> GND
- C6 pad 2: GNDA -> GND
- C7 pad 1: Net-(U5-CLK0) -> /Comb_Generator/CLK1
- C9 pad 1: GNDA -> GND
- D1 pad 1: GNDA -> GND
- D3 pad 1: GNDA -> GND
- J11 pad 1: GNDA -> GND
- J2 pad 1: GNDA -> GND
- RV1 pad 1: GNDA -> GND
- RV2 pad 1: GNDA -> GND
- U13 pad 3: GNDA -> GND
- U2 pad 2: GNDA -> GND
- U5 pad 12: Net-(U5-CLK1) -> unconnected-(U5-CLK1-Pad12)
- U5 pad 13: Net-(U5-CLK0) -> /Comb_Generator/CLK0
- U5 pad 15: unconnected-(U5-CLK7-Pad15) -> /Comb_Generator/CLK1
- U6 pad 2: GNDA -> GND
- U7 pad 3: GNDA -> GND
Routing:
- net +9VA: track 8.74 -> 99.7 mm, vias 0 -> 4
- net +3V3: track 14.1 -> 80.7 mm, vias 0 -> 4
- net /Comb_Generator/10MHz_IN: track 2.67 -> 62.4 mm
- net GND: track 0.86 -> 47.4 mm, vias 1 -> 181
- net /Comb_Generator/CLK0: track 0.00 -> 32.4 mm
- net Net-(C35-Pad1): track 0.00 -> 29.0 mm, vias 0 -> 2
- net /Controller/3V3D_FIL: track 18.2 -> 46.9 mm, vias 0 -> 3
- net /Controller/MISO: track 7.93 -> 31.5 mm
- net /Controller/SCK: track 10.3 -> 33.9 mm
- net Net-(C26-Pad1): track 0.00 -> 18.7 mm
- net /Controller/MOSI: track 10.3 -> 29.0 mm
- net /Comb_Generator/3V3D: track 15.9 -> 33.9 mm, vias 0 -> 2
- net /Comb_Generator/comb_out_1: track 0.00 -> 14.4 mm
- net /Comb_Generator/CLK1: track 0.00 -> 14.0 mm
- net Net-(J5-Pin_6): track 6.92 -> 19.5 mm
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- added copper zone on B.Cu, net GND
- added copper zone on F.Cu, net GND
- added copper zone on In1.Cu, net GND
- added copper zone on In2.Cu, net GND

Commit message: es wird fast fertig...
Parts:
- moved C6 19.0 mm to (175.2, 70.6), turned to 90 degrees
- moved R12 16.1 mm to (177.2, 70.6), turned to -90 degrees
- moved RV1 10.3 mm to (181.4, 70.7), turned to 180 degrees
- moved R13 6.89 mm to (187.6, 69.9), turned to -90 degrees
- moved C50 6.76 mm to (179.5, 58.3), turned to 90 degrees
- moved C5 6.44 mm to (185.7, 58.3), turned to 90 degrees
- moved C32 5.91 mm to (185.7, 69.9)
- moved C7 5.73 mm to (173.4, 65.1)
- moved C25 5.67 mm to (176.3, 66.0)
- moved C26 5.38 mm to (181.6, 58.3), turned to 90 degrees
- moved L2 5.36 mm to (190.4, 65.0)
- moved L3 5.36 mm to (196.2, 65.0)
- moved C9 5.36 mm to (193.2, 66.0)
- moved D1 5.36 mm to (199.0, 66.0)
- moved L1 5.36 mm to (183.8, 62.1)
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Routing:
- net GND: track 47.4 -> 113.3 mm, vias 181 -> 781
- net /Comb_Generator/CLK1: track 14.0 -> 29.4 mm
- net Net-(C26-Pad1): track 18.7 -> 28.6 mm, vias 0 -> 2
- net +9VA: track 99.7 -> 95.0 mm
- net /Comb_Generator/comb_out_1: track 14.4 -> 10.6 mm
- net Net-(C32-Pad1): track 7.33 -> 4.31 mm
- net Net-(C31-Pad1): track 3.33 -> 1.78 mm
- net /Comb_Generator/CLK0: track 32.4 -> 31.1 mm
Other:
- board text added: "+3V3"
- board text added: "A3/INTR"
- board text added: "A4/SDA"
- board text added: "A5/SCL"
- board text added: "D10"
- board text added: "D11/MOSI"
- board text added: "D12/MISO"
- board text added: "D13/SCK"
- board text added: "D8"
- board text added: "D9"
- board text added: "GND"
